File: Camping-LightRelay.kicad_pcb (KiCad board)
At the start: 2 copper layers, 58 x 63 mm, 91 parts, among them CN1 U262-061N-4BVC11, CN101 XHP-2, CN2 907-152A1022D10200, CN3 907-152A1022D10200, CN4 B2B-XH-A, Q1 FDV301N, Q2 BC817, Q3 IRF7404, Q4 BSS138, U1 USBLC6-2SC6, U2 CD4011UBM, U3 SI1865DDL, U4 ME2108A50M, U5 TLC555DTR, U6 LMV358ID

Commit message: Исправление диаметров отверстий
Отверстия пропускания кабеля датчика освещенности слишком малы. Увеличено до 3.5мм
Parts:
- removed the HOLE101 at (131.5, 87.0)
- added HOLE102: MountingHole_3.5mm, MountingHole:MountingHole_3.5mm, F.Cu at (131.5, 87.2)
- HOLE101: value MountingHole_2.1mm -> MountingHole_3.5mm; footprint MountingHole:MountingHole_2.1mm -> MountingHole:MountingHole_3.5mm
- MH1 (x3), MH3: value MountingHole_2.5mm -> MountingHole_2.7mm_M2.5; footprint MountingHole:MountingHole_2.5mm -> MountingHole:MountingHole_2.7mm_M2.5
Changed lines of the file:
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@@
 		)
 	)
-	(footprint "MountingHole:MountingHole_2.5mm"
+	(footprint "MountingHole:MountingHole_2.7mm_M2.5"
 		(layer "F.Cu")
 		(at 123 46)
-		(descr "Mounting Hole 2.5mm, no annular")
-		(tags "mounting hole 2.5mm no annular")
+		(descr "Mounting Hole 2.7mm, no annular, M2.5")
+		(tags "mounting hole 2.7mm no annular m2.5")
 		(property "Reference" "MH1"
 			(at 0 -3.5 0)
@@
 			)
 		)
-		(property "Value" "MountingHole_2.5mm"
+		(property "Value" "MountingHole_2.7mm_M2.5"
 			(at 0 3.5 0)
 			(layer "F.Fab")
@@
 			)
 		)
-		(property "Footprint" "MountingHole:MountingHole_2.5mm"
+		(property "Footprint" "MountingHole:MountingHole_2.7mm_M2.5"
 			(at 0 0 0)
 			(unlocked yes)
@@
 			)
 		)
-		(attr board_only exclude_from_pos_files exclude_from_bom)
+		(attr exclude_from_pos_files exclude_from_bom allow_missing_courtyard)
 		(fp_circle
 			(center 0 0)
-			(end 2.5 0)
+			(end 2.7 0)
 			(stroke
 				(width 0.15)
@@
 		(fp_circle
 			(center 0 0)
-			(end 2.75 0)
+			(end 2.95 0)
 			(stroke
 				(width 0.05)
@@
 		(pad "" np_thru_hole circle
 			(at 0 0)
-			(size 2.5 2.5)
-			(drill 2.5)
+			(size 2.7 2.7)
+			(drill 2.7)
 			(layers "*.Cu" "*.Mask")
 		)
 	)
-	(footprint "MountingHole:MountingHole_2.5mm"
+	(footprint "MountingHole:MountingHole_2.7mm_M2.5"
 		(layer "F.Cu")
 		(at 82 103)
-		(descr "Mounting Hole 2.5mm, no annular")
-		(tags "mounting hole 2.5mm no annular")
+		(descr "Mounting Hole 2.7mm, no annular, M2.5")
+		(tags "mounting hole 2.7mm no annular m2.5")
 		(property "Reference" "MH3"
 			(at 0 -3.5 0)
@@
 			)
 		)
-		(property "Value" "MountingHole_2.5mm"
+		(property "Value" "MountingHole_2.7mm_M2.5"
 			(at 0 3.5 0)
 			(layer "F.Fab")
@@
 			)
 		)
-		(property "Footprint" "MountingHole:MountingHole_2.5mm"
+		(property "Footprint" "MountingHole:MountingHole_2.7mm_M2.5"
 			(at 0 0 0)
 			(unlocked yes)
@@
 			)
 		)
-		(attr board_only exclude_from_pos_files exclude_from_bom)
+		(attr exclude_from_pos_files exclude_from_bom allow_missing_courtyard)
 		(fp_circle
 			(center 0 0)
-			(end 2.5 0)
+			(end 2.7 0)
 			(stroke
 				(width 0.15)
@@
 		(fp_circle
 			(center 0 0)
-			(end 2.75 0)
+			(end 2.95 0)
 			(stroke
 				(width 0.05)
@@
 		(pad "" np_thru_hole circle
 			(at 0 0)
-			(size 2.5 2.5)
-			(drill 2.5)
+			(size 2.7 2.7)
+			(drill 2.7)
 			(layers "*.Cu" "*.Mask")
 		)
@@
 		)
 	)
-	(footprint "MountingHole:MountingHole_2.1mm"
-		(layer "F.Cu")
-		(at 131.5 87)
-		(descr "Mounting Hole 2.1mm, no annular")
-		(tags "mounting hole 2.1mm no annular")
-		(property "Reference" "HOLE101"
-			(at 0 -3.2 0)
-			(layer "F.SilkS")
-			(hide yes)
-			(effects
-				(font
-					(size 1 1)
-					(thickness 0.15)
-				)
-			)
-		)
-		(property "Value" "MountingHole_2.1mm"
-			(at 0 3.2 0)
-			(layer "F.Fab")
-			(hide yes)
-			(effects
-				(font
-					(size 1 1)
-					(thickness 0.15)
-				)
-			)
-		)
-		(property "Footprint" "MountingHole:MountingHole_2.1mm"
-			(at 0 0 0)
-			(unlocked yes)
-			(layer "F.Fab")
-			(hide yes)
-			(effects
-				(font
-					(size 1.27 1.27)
-					(thickness 0.15)
-				)
-			)
-		)
-		(property "Datasheet" ""
-			(at 0 0 0)
-			(unlocked yes)
-			(layer "F.Fab")
-			(hide yes)
-			(effects
-				(font
-					(size 1.27 1.27)
-					(thickness 0.15)
-				)
-			)
-		)
-		(property "Description" ""
-			(at 0 0 0)
-			(unlocked yes)
-			(layer "F.Fab")
-			(hide yes)
-			(effects
-				(font
-					(size 1.27 1.27)
-					(thickness 0.15)
-				)
-			)
-		)
-		(attr exclude_from_pos_files exclude_from_bom)
-		(fp_circle
-			(center 0 0)
-			(end 2.1 0)
-			(stroke
-				(width 0.15)
-				(type solid)
-			)
-			(fill none)
-			(layer "Cmts.User")
-		)
-		(fp_circle
-			(center 0 0)
-			(end 2.35 0)
-			(stroke
-				(width 0.05)
-				(type solid)
-			)
-			(fill none)
-			(layer "F.CrtYd")
-		)
-		(fp_text user "${REFERENCE}"
-			(at 0 0 0)
-			(layer "F.Fab")
-			(effects
-				(font
-					(size 1 1)
-					(thickness 0.15)
-				)
-			)
-		)
-		(pad "" np_thru_hole circle
-			(at 0 0)
-			(size 2.1 2.1)
-			(drill 2.1)
-			(layers "*.Cu" "*.Mask")
-		)
-	)
 	(footprint "PCM_Ferrite_THT_AKL:Ferrite_L8.0mm_D3.5mm_P3.81mm_Vertical"
 		(layer "F.Cu")
@@
 		)
 	)
-	(footprint "MountingHole:MountingHole_2.1mm"
+	(footprint "MountingHole:MountingHole_3.5mm"
 		(layer "F.Cu")
 		(at 131.5 81)
-		(descr "Mounting Hole 2.1mm, no annular")
-		(tags "mounting hole 2.1mm no annular")
+		(descr "Mounting Hole 3.5mm")
 		(property "Reference" "HOLE101"
-			(at 0 -3.2 0)
+			(at 0 -4.5 0)
 			(layer "F.SilkS")
 			(hide yes)
@@
 			)
 		)
-		(property "Value" "MountingHole_2.1mm"
-			(at 0 3.2 0)
+		(property "Value" "MountingHole_3.5mm"
+			(at 0 4.5 0)
 			(layer "F.Fab")
 			(hide yes)
@@
 			)
 		)
-		(property "Footprint" "MountingHole:MountingHole_2.1mm"
+		(property "Footprint" "MountingHole:MountingHole_3.5mm"
 			(at 0 0 0)
 			(unlocked yes)
@@
 		)
 		(attr exclude_from_pos_files exclude_from_bom)
-		(fp_circle
-			(center 0 0)
-			(end 2.1 0)
-			(stroke
-				(width 0.15)
-				(type solid)
-			)
-			(fill none)
-			(layer "Cmts.User")
-		)
-		(fp_circle
-			(center 0 0)
-			(end 2.35 0)
-			(stroke
-				(width 0.05)
-				(type solid)
-			)
-			(fill none)
-			(layer "F.CrtYd")
-		)
 		(fp_text user "${REFERENCE}"
 			(at 0 0 0)
@@
 		(pad "" np_thru_hole circle
 			(at 0 0)
-			(size 2.1 2.1)
-			(drill 2.1)
+			(size 3.5 3.5)
+			(drill 3.5)
 			(layers "*.Cu" "*.Mask")
 		)
@@
 		)
 	)
-	(footprint "MountingHole:MountingHole_2.5mm"
+	(footprint "MountingHole:MountingHole_2.7mm_M2.5"
 		(layer "F.Cu")
 		(at 123 103)
-		(descr "Mounting Hole 2.5mm, no annular")
-		(tags "mounting hole 2.5mm no annular")
+		(descr "Mounting Hole 2.7mm, no annular, M2.5")
+		(tags "mounting hole 2.7mm no annular m2.5")
 		(property "Reference" "MH1"
 			(at 0 -3.5 0)
@@
 			)
 		)
-		(property "Value" "MountingHole_2.5mm"
+		(property "Value" "MountingHole_2.7mm_M2.5"
 			(at 0 3.5 0)
 			(layer "F.Fab")
@@
 			)
 		)
-		(property "Footprint" "MountingHole:MountingHole_2.5mm"
+		(property "Footprint" "MountingHole:MountingHole_2.7mm_M2.5"
 			(at 0 0 0)
 			(unlocked yes)
@@
 			)
 		)
-		(attr board_only exclude_from_pos_files exclude_from_bom)
+		(attr exclude_from_pos_files exclude_from_bom allow_missing_courtyard)
 		(fp_circle
 			(center 0 0)
-			(end 2.5 0)
+			(end 2.7 0)
 			(stroke
 				(width 0.15)
@@
 		(fp_circle
 			(center 0 0)
-			(end 2.75 0)
+			(end 2.95 0)
 			(stroke
 				(width 0.05)
@@
 		(pad "" np_thru_hole circle
 			(at 0 0)
-			(size 2.5 2.5)
-			(drill 2.5)
+			(size 2.7 2.7)
+			(drill 2.7)
 			(layers "*.Cu" "*.Mask")
 		)
 	)
-	(footprint "MountingHole:MountingHole_2.5mm"
+	(footprint "MountingHole:MountingHole_2.7mm_M2.5"
 		(layer "F.Cu")
 		(at 82 46)
-		(descr "Mounting Hole 2.5mm, no annular")
-		(tags "mounting hole 2.5mm no annular")
+		(descr "Mounting Hole 2.7mm, no annular, M2.5")
+		(tags "mounting hole 2.7mm no annular m2.5")
 		(property "Reference" "MH1"
 			(at 0 -3.5 0)
@@
 			)
 		)
-		(property "Value" "MountingHole_2.5mm"
+		(property "Value" "MountingHole_2.7mm_M2.5"
 			(at 0 3.5 0)
 			(layer "F.Fab")
@@
 			)
 		)
-		(property "Footprint" "MountingHole:MountingHole_2.5mm"
+		(property "Footprint" "MountingHole:MountingHole_2.7mm_M2.5"
 			(at 0 0 0)
 			(unlocked yes)
@@
 			)
 		)
-		(attr board_only exclude_from_pos_files exclude_from_bom)
+		(attr exclude_from_pos_files exclude_from_bom allow_missing_courtyard)
 		(fp_circle
 			(center 0 0)
-			(end 2.5 0)
+			(end 2.7 0)
 			(stroke
 				(width 0.15)
@@
 		(fp_circle
 			(center 0 0)
-			(end 2.75 0)
+			(end 2.95 0)
 			(stroke
 				(width 0.05)
@@
 		(pad "" np_thru_hole circle
 			(at 0 0)
-			(size 2.5 2.5)
-			(drill 2.5)
+			(size 2.7 2.7)
+			(drill 2.7)
 			(layers "*.Cu" "*.Mask")
 		)
@@
 		)
 	)
+	(footprint "MountingHole:MountingHole_3.5mm"
+		(layer "F.Cu")
+		(at 131.5 87.25)
+		(descr "Mounting Hole 3.5mm")
+		(property "Reference" "HOLE102"
+			(at 0 -4.5 0)
+			(layer "F.SilkS")
+			(hide yes)
+			(effects
+				(font
+					(size 1 1)
+					(thickness 0.15)
+				)
+			)
+		)
+		(property "Value" "MountingHole_3.5mm"
+			(at 0 4.5 0)
+			(layer "F.Fab")
+			(hide yes)
+			(effects
+				(font
+					(size 1 1)
+					(thickness 0.15)
+				)
+			)
+		)
+		(property "Footprint" "MountingHole:MountingHole_3.5mm"
+			(at 0 0 0)
+			(unlocked yes)
+			(layer "F.Fab")
+			(hide yes)
+			(effects
+				(font
+					(size 1.27 1.27)
+					(thickness 0.15)
+				)
+			)
+		)
+		(property "Datasheet" ""
+			(at 0 0 0)
+			(unlocked yes)
+			(layer "F.Fab")
+			(hide yes)
+			(effects
+				(font
+					(size 1.27 1.27)
+					(thickness 0.15)
+				)
+			)
+		)
+		(property "Description" ""
+			(at 0 0 0)
+			(unlocked yes)
+			(layer "F.Fab")
+			(hide yes)
+			(effects
+				(font
+					(size 1.27 1.27)
+					(thickness 0.15)
+				)
+			)
+		)
+		(attr exclude_from_pos_files exclude_from_bom)
+		(fp_text user "${REFERENCE}"
+			(at 0 0 0)
+			(layer "F.Fab")
+			(effects
+				(font
+					(size 1 1)
+					(thickness 0.15)
+				)
+			)
+		)
+		(pad "" np_thru_hole circle
+			(at 0 0)
+			(size 3.5 3.5)
+			(drill 3.5)
+			(layers "*.Cu" "*.Mask")
+		)
+	)
