File: Camping-LightRelay.kicad_sch (KiCad schematic)
At the start: 57 parts, among them CN1 U262-061N-4BVC11, CN2 907-152A1022D10200, CN3 907-152A1022D10200, Q1 FDV301N, Q2 BC817, Q3 IRF7404, U1 USBLC6-2SC6, U2 CD4011UBM, U3 SI1865DDL, U4 ME2108A50M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

Commit message: Мелкий рефакторинг
- Обновление Readme.md
- Правки в печатную плату
- Переименование сигналов
- добавление исключений в .gitignore
Parts:
- C4: value 100uFx10V -> 10uFx16V; footprint Capacitor_Tantalum_SMD:CP_EIA-3528-15_AVX-H_Pad1.50x2.35mm_HandSolder -> Capacitor_Tantalum_SMD:CP_EIA-3216-12_Kemet-S_Pad1.58x1.35mm_HandSolder
- R10: value 470 -> 560
- R3: footprint Resistor_THT:R_Axial_DIN0309_L9.0mm_D3.2mm_P5.08mm_Vertical -> PCM_Resistor_THT_AKL:R_Axial_DIN0309_L9.0mm_D3.2mm_P2.54mm_Vertical
Other:
- sheet Субмодуль фотореле ports: added ~{OUT}; removed ~{RELAY_ON}
- moved on the sheet: R9, U2A, U2B
Changed lines of the file:
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@@
 	)
 	(junction
-		(at 139.7 153.67)
-		(diameter 0)
-		(color 0 0 0 0)
-	)
-	(junction
 		(at 105.41 29.21)
 		(diameter 0)
@@
 	)
 	(junction
-		(at 121.92 156.21)
+		(at 119.38 156.21)
 		(diameter 0)
 		(color 0 0 0 0)
@@
 	)
 	(junction
+		(at 139.7 158.75)
+		(diameter 0)
+		(color 0 0 0 0)
+	)
+	(junction
+		(at 137.16 153.67)
+		(diameter 0)
+		(color 0 0 0 0)
+	)
+	(junction
 		(at 220.98 137.16)
 		(diameter 0)
@@
 	)
 	(junction
-		(at 139.7 158.75)
-		(diameter 0)
-		(color 0 0 0 0)
-	)
-	(junction
 		(at 129.54 49.53)
 		(diameter 0)
@@
 	(wire
 		(pts
+			(xy 139.7 158.75) (xy 157.48 158.75)
+		)
+		(stroke
+			(width 0)
+			(type default)
+		)
+	)
+	(wire
+		(pts
 			(xy 175.26 41.91) (xy 175.26 29.21)
 		)
@@
 	(wire
 		(pts
-			(xy 121.92 153.67) (xy 121.92 156.21)
+			(xy 119.38 153.67) (xy 119.38 156.21)
 		)
 		(stroke
@@
 	(wire
 		(pts
+			(xy 137.16 153.67) (xy 142.24 153.67)
+		)
+		(stroke
+			(width 0)
+			(type default)
+		)
+	)
+	(wire
+		(pts
 			(xy 35.56 63.5) (xy 58.42 63.5)
 		)
@@
 	(wire
 		(pts
-			(xy 139.7 158.75) (xy 157.48 158.75)
+			(xy 134.62 158.75) (xy 139.7 158.75)
 		)
 		(stroke
@@
 	(wire
 		(pts
-			(xy 137.16 153.67) (xy 139.7 153.67)
+			(xy 134.62 153.67) (xy 137.16 153.67)
 		)
 		(stroke
@@
 	(wire
 		(pts
+			(xy 139.7 140.97) (xy 139.7 158.75)
+		)
+		(stroke
+			(width 0)
+			(type default)
+		)
+	)
+	(wire
+		(pts
 			(xy 228.6 124.46) (xy 228.6 151.13)
 		)
@@
 	(wire
 		(pts
-			(xy 121.92 156.21) (xy 121.92 158.75)
+			(xy 119.38 156.21) (xy 119.38 158.75)
 		)
 		(stroke
@@
 	(wire
 		(pts
-			(xy 101.6 156.21) (xy 106.68 156.21)
+			(xy 101.6 156.21) (xy 104.14 156.21)
 		)
 		(stroke
@@
 	(wire
 		(pts
-			(xy 139.7 137.16) (xy 139.7 153.67)
+			(xy 137.16 137.16) (xy 137.16 153.67)
 		)
 		(stroke
@@
 	(wire
 		(pts
-			(xy 137.16 158.75) (xy 139.7 158.75)
-		)
-		(stroke
-			(width 0)
-			(type default)
-		)
-	)
-	(wire
-		(pts
 			(xy 154.94 29.21) (xy 156.21 29.21)
 		)
@@
 	(wire
 		(pts
-			(xy 139.7 153.67) (xy 142.24 153.67)
-		)
-		(stroke
-			(width 0)
-			(type default)
-		)
-	)
-	(wire
-		(pts
 			(xy 212.09 22.86) (xy 184.15 22.86)
 		)
@@
 	(wire
 		(pts
-			(xy 139.7 158.75) (xy 139.7 162.56)
-		)
-		(stroke
-			(width 0)
-			(type default)
-		)
-	)
-	(wire
-		(pts
-			(xy 128.27 137.16) (xy 139.7 137.16)
+			(xy 128.27 137.16) (xy 137.16 137.16)
 		)
 		(stroke
@@
 	)
 	(rectangle
-		(start 107.315 144.145)
-		(end 137.795 160.655)
+		(start 104.775 144.145)
+		(end 135.255 160.655)
 		(stroke
 			(width 0)
@@
 	)
 	(rectangle
+		(start 137.795 132.715)
+		(end 147.32 140.97)
+		(stroke
+			(width 0)
+			(type dash)
+		)
+		(fill
+			(type none)
+		)
+	)
+	(rectangle
 		(start 149.225 33.655)
 		(end 161.29 59.69)
@@
 	(text "AND"
 		(exclude_from_sim no)
-		(at 122.428 148.082 0)
+		(at 119.888 148.082 0)
 		(effects
 			(font
@@
 		)
 	)
+	(text "Optional"
+		(exclude_from_sim yes)
+		(at 149.352 140.97 90)
+		(effects
+			(font
+				(size 1.27 1.27)
+			)
+			(justify left bottom)
+		)
+	)
 	(label "SH-NET"
 		(at 25.4 63.5 90)
@@
 			)
 		)
-		(property "Description" "Littelfuse axial lead 3.6x10 mm"
+		(property "Description" "SMD Fuse"
 			(at 53.34 29.21 0)
 			(effects
@@
 	(symbol
 		(lib_id "4xxx:4011")
-		(at 114.3 156.21 0)
+		(at 111.76 156.21 0)
 		(mirror y)
 		(unit 1)
@@
 		(dnp no)
 		(property "Reference" "U2"
-			(at 114.3083 147.32 0)
+			(at 111.7683 147.32 0)
 			(effects
 				(font
@@
 		)
 		(property "Value" "CD4011UBM"
-			(at 114.3083 149.86 0)
+			(at 111.7683 149.86 0)
 			(effects
 				(font
@@
 		)
 		(property "Footprint" "Package_SO:SOIC-14_3.9x8.7mm_P1.27mm"
-			(at 114.3 156.21 0)
+			(at 111.76 156.21 0)
 			(effects
 				(font
@@
 		)
 		(property "Datasheet" "http://www.intersil.com/content/dam/Intersil/documents/cd40/cd4011bms-12bms-23bms.pdf"
-			(at 114.3 156.21 0)
+			(at 111.76 156.21 0)
 			(effects
 				(font
@@
 		)
 		(property "Description" "Quad Nand 2 inputs"
-			(at 114.3 156.21 0)
+			(at 111.76 156.21 0)
 			(effects
 				(font
@@
 			)
 		)
-		(property "Value" "470"
+		(property "Value" "560"
 			(at 156.464 38.862 0)
 			(effects
@@
 			)
 		)
-		(property "Footprint" "Resistor_THT:R_Axial_DIN0309_L9.0mm_D3.2mm_P5.08mm_Vertical"
+		(property "Footprint" "PCM_Resistor_THT_AKL:R_Axial_DIN0309_L9.0mm_D3.2mm_P2.54mm_Vertical"
 			(at 90.932 36.83 90)
 			(effects
@@
 	(symbol
 		(lib_id "4xxx:4011")
-		(at 129.54 156.21 0)
+		(at 127 156.21 0)
 		(mirror y)
 		(unit 2)
@@
 		(dnp no)
 		(property "Reference" "U2"
-			(at 129.5483 147.32 0)
+			(at 127.0083 147.32 0)
 			(effects
 				(font
@@
 		)
 		(property "Value" "CD4011UBM"
-			(at 129.5483 149.86 0)
+			(at 127.0083 149.86 0)
 			(effects
 				(font
@@
 		)
 		(property "Footprint" "Package_SO:SOIC-14_3.9x8.7mm_P1.27mm"
-			(at 129.54 156.21 0)
+			(at 127 156.21 0)
 			(effects
 				(font
@@
 		)
 		(property "Datasheet" "http://www.intersil.com/content/dam/Intersil/documents/cd40/cd4011bms-12bms-23bms.pdf"
-			(at 129.54 156.21 0)
+			(at 127 156.21 0)
 			(effects
 				(font
@@
 		)
 		(property "Description" "Quad Nand 2 inputs"
-			(at 129.54 156.21 0)
+			(at 127 156.21 0)
 			(effects
 				(font
@@
 	(symbol
 		(lib_id "Device:R")
-		(at 139.7 166.37 0)
+		(at 139.7 137.16 180)
 		(unit 1)
 		(exclude_from_sim no)
@@
 		(on_board yes)
 		(dnp no)
-		(fields_autoplaced yes)
 		(property "Reference" "R9"
-			(at 142.24 165.0999 0)
+			(at 141.732 136.652 0)
 			(effects
 				(font
 					(size 1.27 1.27)
 				)
-				(justify left)
+				(justify right top)
 			)
 		)
 		(property "Value" "100k"
-			(at 142.24 167.6399 0)
+			(at 141.732 137.16 0)
 			(effects
 				(font
 					(size 1.27 1.27)
 				)
-				(justify left)
+				(justify right bottom)
 			)
 		)
 		(property "Footprint" "PCM_Resistor_SMD_AKL:R_0603_1608Metric_Pad0.98x0.95mm"
-			(at 137.922 166.37 90)
+			(at 141.478 137.16 90)
 			(effects
 				(font
@@
 		)
 		(property "Datasheet" "~"
-			(at 139.7 166.37 0)
+			(at 139.7 137.16 0)
 			(effects
 				(font
@@
 		)
 		(property "Description" "Resistor"
-			(at 139.7 166.37 0)
+			(at 139.7 137.16 0)
 			(effects
 				(font
@@
 	(symbol
 		(lib_id "power:VCC")
-		(at 139.7 170.18 180)
+		(at 139.7 133.35 0)
 		(unit 1)
 		(exclude_from_sim no)
@@
 		(on_board yes)
 		(dnp no)
-		(fields_autoplaced yes)
 		(property "Reference" "#PWR05"
-			(at 139.7 166.37 0)
+			(at 139.7 137.16 0)
 			(effects
 				(font
@@
 		)
 		(property "Value" "VCC"
-			(at 139.7 175.26 0)
+			(at 139.7 130.302 0)
 			(effects
 				(font
 					(size 1.27 1.27)
 				)
+				(justify bottom)
 			)
 		)
 		(property "Footprint" ""
-			(at 139.7 170.18 0)
+			(at 139.7 133.35 0)
 			(effects
 				(font
@@
 		)
 		(property "Datasheet" ""
-			(at 139.7 170.18 0)
+			(at 139.7 133.35 0)
 			(effects
 				(font
@@
 		)
 		(property "Description" "Power symbol creates a global label with name \"VCC\""
-			(at 139.7 170.18 0)
+			(at 139.7 133.35 0)
 			(effects
 				(font
@@
 			)
 		)
-		(property "Value" "100uFx10V"
+		(property "Value" "10uFx16V"
 			(at 143.002 51.308 0)
 			(effects
@@
 			)
 		)
-		(property "Footprint" "Capacitor_Tantalum_SMD:CP_EIA-3528-15_AVX-H_Pad1.50x2.35mm_HandSolder"
+		(property "Footprint" "Capacitor_Tantalum_SMD:CP_EIA-3216-12_Kemet-S_Pad1.58x1.35mm_HandSolder"
 			(at 144.4752 49.53 0)
 			(effects
@@
 			)
 		)
-		(pin "~{RELAY_ON}" output
+		(pin "~{OUT}" output
 			(at 238.76 72.39 180)
 			(effects

Commit message: Обновление перед публикацией
- Удаление лишнего файла симуляции
- Рефакторинг электрической схемы и печатной платой.
- Добавление файла симуляции разряда ионистора.
- Удаление лишних захламляющих файлов
- Рефакторинг симуляции схем
- Обновление описания Readme
Other:
- title: Высокочувствительное фотореле с микропотреблением -> Модуль периферии. Схема ЭП.
Changed lines of the file:
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@@
 	(paper "A4")
 	(title_block
-		(title "Высокочувствительное фотореле с микропотреблением")
+		(title "Модуль периферии. Схема ЭП.")
 		(date "2024-05-12")
-		(rev "1.0")
-		(comment 1 "Э04.01.01 Э3")
+		(rev "1.3")
+		(comment 1 "ФРК.42126.002-03 Э3")
 		(comment 2 "В.Иншаков")
+		(comment 7 "Э04.01.01 Э3")
 	)
 	(junction

Commit message: Изменение номинала резистора R3
Возможна нестабильная работа запуска PowerBank-ов при номинале *47 Ом*. Уменьшено до *43* Ом, чтобы ток составлял _100мА_
Parts:
- R3: value 47 1W -> 43 1W
Changed lines of the file:
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@@
 			)
 		)
-		(property "Value" "47 1W"
+		(property "Value" "43 1W"
 			(at 94.742 37.084 0)
 			(effects
